Commit message: feat: use seven-cylinder foot collisions in C1 URDF and MuJoCo models

File: urdf/walker_c1.urdf (robot description, URDF)
Before this commit: robot walker_c1_description, 40 links, 39 joints
Links:
- link L_ankle_roll_link: geometry collision cylinder length=0.06 radius=0.012; collision cylinder length=0.06 radius=0.012
- link R_ankle_roll_link: geometry collision cylinder length=0.06 radius=0.012; collision cylinder length=0.06 radius=0.012

File: urdf/walker_c1_with_dummyhands.urdf (robot description, URDF)
Before this commit: robot walker_c1_description_with_dummy_hands, 42 links, 41 joints
Links:
- link L_ankle_roll_link: geometry collision cylinder length=0.06 radius=0.012; collision cylinder length=0.06 radius=0.012
- link R_ankle_roll_link: geometry collision cylinder length=0.06 radius=0.012; collision cylinder length=0.06 radius=0.012

File: urdf/walker_c1_with_hands.urdf (robot description, URDF)
Before this commit: robot walker_c1_description_with_hands, 66 links, 65 joints
Links:
- link L_ankle_roll_link: geometry collision cylinder length=0.06 radius=0.012; collision cylinder length=0.06 radius=0.012
- link R_ankle_roll_link: geometry collision cylinder length=0.06 radius=0.012; collision cylinder length=0.06 radius=0.012
